Commit message: Added first draft of tutorial

File: urdf/robot_model.xacro (robot description, xacro)
@@ -1,12 +1,12 @@
 <?xml version='1.0'?>
 <robot name="robot_model" xmlns:xacro="http://www.ros.org/wiki/xacro">
-  <xacro:include filename="$(find object_follower)/urdf/robot_model.gazebo" />
+  <xacro:include filename="$(find ros_tutorial)/urdf/robot_model.gazebo" />
   <link name="robot_footprint"></link>
   <gazebo reference="chassis">
-    <material>Gazebo/Blue</material>
+    <material>Gazebo/Orange</material>
   </gazebo>
   <gazebo reference="front_caster">
     <selfCollide>false</selfCollide>
-    <material>Gazebo/White</material>
+    <material>Gazebo/Black</material>
     <mu1>0</mu1>
     <mu2>0</mu2>
@@ -16,5 +16,5 @@
   <gazebo reference="back_caster">
     <selfCollide>false</selfCollide>
-    <material>Gazebo/White</material>
+    <material>Gazebo/Black</material>
     <mu1>0</mu1>
     <mu2>0</mu2>
@@ -23,12 +23,12 @@
   </gazebo>
   <gazebo reference="right_pad">
-    <material>Gazebo/Blue</material>
+    <material>Gazebo/Orange</material>
   </gazebo>
   <gazebo reference="left_pad">
-    <material>Gazebo/Blue</material>
+    <material>Gazebo/Orange</material>
   </gazebo>
   <gazebo reference="left_wheel">
     <selfCollid>false</selfCollid>
-    <material>Gazebo/White</material>
+    <material>Gazebo/Black</material>
     <mu1>10</mu1>
     <mu2>10</mu2>
@@ -38,5 +38,5 @@
   <gazebo reference="right_wheel">
     <selfCollid>false</selfCollid>
-    <material>Gazebo/White</material>
+    <material>Gazebo/Black</material>
     <mu1>10</mu1>
     <mu2>10</mu2>
@@ -229,10 +229,9 @@
     <axis xyz="0 1 0" rpy="0 0 0"/>
   </joint>
-  <!-- CAMERA AIR LINK -->
-  <link name="camera_air">
-    <pose>0 0 0 0 0 0</pose>
-    <inertial>
-      <mass value="0"/>
-      <origin xyz="0.0 0.0 0.0" rpy="0 0 0"/>
+  <link name="right_pad">
+    <pose>0 0 0 0 0 0</pose>
+    <inertial>
+      <mass value="0.1"/>
+      <origin xyz="0 0 0" rpy="0 0 0"/>
       <inertia
               ixx="1e-6" ixy="0" ixz="0"
@@ -241,24 +240,24 @@
       />
     </inertial>
-    <visual name='camera_air_visual'>
-      <origin xyz="0 0 0" rpy=" 0 0 0"/>
-      <geometry>
-        <box size="0.001 0.001 0.001"/>
-      </geometry>
-    </visual>
-    <collision name='camera_air_collision'>
-      <origin xyz="0 0 0" rpy=" 0 0 0"/>
-      <geometry>
-        <box size="0.0 0.0 0.0"/>
-      </geometry>
-    </collision>
-  </link>
-  <joint type="fixed" name="camera_air_joint">
-    <origin xyz="0.2 0.0 2.0" rpy="0 1.5707 0"/>
-    <child link="camera_air"/>
-    <parent link="chassis"/>
-    <axis xyz="0 1 0" rpy="0 0 0"/>
-  </joint>
-  <link name="right_pad">
+    <visual name='right_pad_visual'>
+      <origin xyz="0 0 0" rpy=" 0 0 0"/>
+      <geometry>
+        <box size="0.06 0.06 0.1"/>
+      </geometry>
+    </visual>
+    <collision name='right_pad_collision'>
+      <origin xyz="0 0 0" rpy=" 0 0 0"/>
+      <geometry>
+        <box size="0.06 0.06 0.1"/>
+      </geometry>
+    </collision>
+  </link>
+  <joint type="fixed" name="right_pad_joint">
+    <origin xyz="-0.17 -0.13 0" rpy="0 0 0"/>
+    <child link="right_pad"/>
+    <parent link="chassis"/>
+    <axis xyz="0 1 0" rpy="0 0 0"/>
+  </joint>
+  <link name="left_pad">
     <pose>0 0 0 0 0 0</pose>
     <inertial>
@@ -271,5 +270,5 @@
       />
     </inertial>
-    <visual name='right_pad_visual'>
+    <visual name='left_pad_visual'>
       <origin xyz="0 0 0" rpy=" 0 0 0"/>
       <geometry>
@@ -277,5 +276,5 @@
       </geometry>
     </visual>
-    <collision name='right_pad_collision'>
+    <collision name='left_pad_collision'>
       <origin xyz="0 0 0" rpy=" 0 0 0"/>
       <geometry>
@@ -284,14 +283,14 @@
     </collision>
   </link>
-  <joint type="fixed" name="right_pad_joint">
-    <origin xyz="-0.17 -0.13 0" rpy="0 0 0"/>
-    <child link="right_pad"/>
-    <parent link="chassis"/>
-    <axis xyz="0 1 0" rpy="0 0 0"/>
-  </joint>
-  <link name="left_pad">
-    <pose>0 0 0 0 0 0</pose>
-    <inertial>
-      <mass value="0.1"/>
+  <joint type="fixed" name="left_pad_joint">
+    <origin xyz="-0.17 0.13 0" rpy="0 0 0"/>
+    <child link="left_pad"/>
+    <parent link="chassis"/>
+    <axis xyz="0 1 0" rpy="0 0 0"/>
+  </joint>
+  <!-- LIDAR LINK -->
+  <link name="hokuyo">
+    <inertial>
+      <mass value="1e-5"/>
       <origin xyz="0 0 0" rpy="0 0 0"/>
       <inertia
@@ -301,38 +300,8 @@
       />
     </inertial>
-    <visual name='left_pad_visual'>
-      <origin xyz="0 0 0" rpy=" 0 0 0"/>
-      <geometry>
-        <box size="0.06 0.06 0.1"/>
-      </geometry>
-    </visual>
-    <collision name='left_pad_collision'>
-      <origin xyz="0 0 0" rpy=" 0 0 0"/>
-      <geometry>
-        <box size="0.06 0.06 0.1"/>
-      </geometry>
-    </collision>
-  </link>
-  <joint type="fixed" name="left_pad_joint">
-    <origin xyz="-0.17 0.13 0" rpy="0 0 0"/>
-    <child link="left_pad"/>
-    <parent link="chassis"/>
-    <axis xyz="0 1 0" rpy="0 0 0"/>
-  </joint>
-  <!-- LIDAR LINK -->
-  <link name="hokuyo">
-    <inertial>
-      <mass value="1e-5"/>
-      <origin xyz="0 0 0" rpy="0 0 0"/>
-      <inertia
-              ixx="1e-6" ixy="0" ixz="0"
-              iyy="1e-6" iyz="0"
-              izz="1e-6"
-      />
-    </inertial>
     <visual name='hokuyo_visual'>
       <origin xyz="0 0 0" rpy=" 0 0 0"/>
       <geometry>
-        <mesh filename="package://object_follower/meshes/hokuyo.dae"/>
+        <mesh filename="package://ros_tutorial/meshes/hokuyo.dae"/>
       </geometry>
     </visual>
